Commit message: add joints and links

File: src/rrm_cv3_kocur/urdf/arm.urdf (robot description, URDF)
Before this commit: robot arm, 6 links, 5 joints
Links:
- added link joint_3; visual sphere radius=0.03
- added link joint_4; visual sphere radius=0.03
- added link link3; visual cylinder length=0.178 radius=0.01
- added link link4; visual cylinder length=0.178 radius=0.01
Joints:
- removed joint joint_2_to_tool0
- added joint joint_3: type revolute, parent joint_2, child joint_3, origin xyz=0 0 0 rpy=0 0 0, axis 0 0 1, limit lower=-1.62 upper=1.62 effort=1000.0 velocity=0.5
- added joint joint_4: type revolute, parent joint_3, child joint_4, origin xyz=0 0 0 rpy=0 0 0, axis 0 0 1, limit lower=-1.62 upper=1.62 effort=1000.0 velocity=0.5
- added joint joint_4_to_tool0: type fixed, parent joint_4, child tool0, origin xyz=0 0 0.178 rpy=0 0 0
- added joint link3_to_joint_3: type fixed, parent joint_3, child link3, origin xyz=0 0 0.1015 rpy=0 0 0
- added joint link4_to_joint_4: type fixed, parent joint_4, child link4, origin xyz=0 0 0.1015 rpy=0 0 0

Commit message: edit xyz

File: src/rrm_cv3_kocur/urdf/arm.urdf (robot description, URDF)
Before this commit: robot arm, 10 links, 9 joints
Joints:
- joint joint_3: type revolute -> continuous
- joint link3_to_joint_3: origin xyz=0 0 0.1015 rpy=0 0 0 -> xyz=0 0 0.089 rpy=0 0 0
- joint link4_to_joint_4: origin xyz=0 0 0.1015 rpy=0 0 0 -> xyz=0 0 0.089 rpy=0 0 0

Commit message: edit last origin

File: src/rrm_cv3_kocur/urdf/arm.urdf (robot description, URDF)
Before this commit: robot arm, 10 links, 9 joints
Joints:
- joint joint_4_to_tool0: origin xyz=0 0 0.178 rpy=0 0 0 -> xyz=0 0 0.36865 rpy=0 0 0

Commit message: test

File: src/rrm_cv3_kocur/urdf/arm.urdf (robot description, URDF)
Before this commit: robot arm, 10 links, 9 joints
Joints:
- joint joint_4_to_tool0: origin xyz=0 0 0.36865 rpy=0 0 0 -> xyz=0 0 0.7 rpy=0 0 0

Commit message: joint3 type

File: src/rrm_cv3_kocur/urdf/arm.urdf (robot description, URDF)
Before this commit: robot arm, 10 links, 9 joints
Joints:
- joint joint_3: type continuous -> prismatic
- joint joint_4_to_tool0: origin xyz=0 0 0.7 rpy=0 0 0 -> xyz=0 0 0.36865 rpy=0 0 0

Commit message: tool

File: src/rrm_cv3_kocur/urdf/arm.urdf (robot description, URDF)
Before this commit: robot arm, 10 links, 9 joints
Joints:
- joint joint_2: origin xyz=0 0 0.203 rpy=0 0 0 -> xyz=0 0 0 rpy=0 0 0
- joint joint_4: axis 0 0 1 -> 0 1 0
- joint joint_4_to_tool0: origin xyz=0 0 0.36865 rpy=0 0 0 -> xyz=0 0 0 rpy=0 0 0

Commit message: prismatic

File: src/rrm_cv3_kocur/urdf/arm.urdf (robot description, URDF)
Before this commit: robot arm, 10 links, 9 joints
Joints:
- joint link3_to_joint_3: type fixed -> prismatic

Commit message: fixed back

File: src/rrm_cv3_kocur/urdf/arm.urdf (robot description, URDF)
Before this commit: robot arm, 10 links, 9 joints
Joints:
- joint link3_to_joint_3: type prismatic -> fixed

Commit message: tool to joint4

File: src/rrm_cv3_kocur/urdf/arm.urdf (robot description, URDF)
Before this commit: robot arm, 9 links, 9 joints
Links:
- added link base_link; visual cylinder length=0.01 radius=0.05

Commit message: link to joint

File: src/rrm_cv3_kocur/urdf/arm.urdf (robot description, URDF)
Before this commit: robot arm, 10 links, 9 joints
Joints:
- joint joint_3: child joint_3 -> link_3

Commit message: bruh

File: src/rrm_cv3_kocur/urdf/arm.urdf (robot description, URDF)
Before this commit: robot arm, 10 links, 9 joints
Joints:
- joint joint_3: axis 0 0 1 -> 1 1 1; child link_3 -> joint_3

Commit message: prisma

File: src/rrm_cv3_kocur/urdf/arm.urdf (robot description, URDF)
Before this commit: robot arm, 10 links, 9 joints
Joints:
- joint joint_3: axis 1 1 1 -> 0 0 1

Commit message: upper lower

File: src/rrm_cv3_kocur/urdf/arm.urdf (robot description, URDF)
Before this commit: robot arm, 10 links, 9 joints
Joints:
- joint joint_3: limit lower=-1.62 upper=1.62 effort=1000.0 velocity=0.5 -> lower=0 upper=0.089 effort=1000.0 velocity=0.5

Commit message: uprava limit

File: src/rrm_cv3_kocur/urdf/arm.urdf (robot description, URDF)
Before this commit: robot arm, 10 links, 9 joints
Joints:
- joint joint_3: limit lower=0 upper=0.089 effort=1000.0 velocity=0.5 -> lower=0.089 upper=0.0 effort=1000.0 velocity=0.5

Commit message: limits edit

File: src/rrm_cv3_kocur/urdf/arm.urdf (robot description, URDF)
Before this commit: robot arm, 10 links, 9 joints
Joints:
- joint joint_3: limit lower=0.089 upper=0.0 effort=1000.0 velocity=0.5 -> lower=0 upper=-0.96 effort=1000.0 velocity=0.5

Commit message: once more

File: src/rrm_cv3_kocur/urdf/arm.urdf (robot description, URDF)
Before this commit: robot arm, 10 links, 9 joints
Joints:
- joint joint_3: limit lower=0 upper=-0.96 effort=1000.0 velocity=0.5 -> lower=0 upper=0.178 effort=1000.0 velocity=0.5

Commit message: ups

File: src/rrm_cv3_kocur/urdf/arm.urdf (robot description, URDF)
Before this commit: robot arm, 10 links, 9 joints
Joints:
- joint joint_3: limit lower=0 upper=0.178 effort=1000.0 velocity=0.5 -> lower=-0.178 upper=0 effort=1000.0 velocity=0.5

Commit message: link base tool0

File: src/rrm_cv3_kocur/urdf/arm.urdf (robot description, URDF)
Before this commit: robot arm, 10 links, 9 joints
Joints:
- removed joint joint_4_to_tool0
- added joint base_link_to_tool0: type fixed, parent joint_4, child tool0, origin xyz=0 0 0 rpy=0 0 0

Commit message: link base to tool

File: src/rrm_cv3_kocur/urdf/arm.urdf (robot description, URDF)
Before this commit: robot arm, 10 links, 9 joints
Joints:
- joint base_link_to_tool0: parent joint_4 -> base_link

Commit message: cudo

File: src/rrm_cv3_kocur/urdf/arm.urdf (robot description, URDF)
Before this commit: robot arm, 10 links, 9 joints
Joints:
- removed joint base_link_to_tool0

Commit message: zas a raz

File: src/rrm_cv3_kocur/urdf/arm.urdf (robot description, URDF)
Before this commit: robot arm, 10 links, 8 joints
Joints:
- added joint joint_4_to_tool0: type fixed, parent joint_4, child tool0, origin xyz=0 0 0 rpy=0 0 0
- joint joint_3: limit lower=-0.178 upper=0 effort=1000.0 velocity=0.5 -> lower=-0.178 upper=0.178 effort=1000.0 velocity=0.5

Commit message: last joint

File: src/rrm_cv3_kocur/urdf/arm.urdf (robot description, URDF)
Before this commit: robot arm, 10 links, 9 joints
Joints:
- joint joint_3: limit lower=-0.178 upper=0.178 effort=1000.0 velocity=0.5 -> lower=-0.178 upper=0 effort=1000.0 velocity=0.5

Commit message: 203

File: src/rrm_cv3_kocur/urdf/arm.urdf (robot description, URDF)
Before this commit: robot arm, 10 links, 9 joints
Joints:
- joint link1_to_joint_1: origin xyz=0 0 0.1015 rpy=0 0 0 -> xyz=0 0 0.203 rpy=0 0 0

Commit message: 0.0

File: src/rrm_cv3_kocur/urdf/arm.urdf (robot description, URDF)
Before this commit: robot arm, 10 links, 9 joints
Joints:
- joint link1_to_joint_1: origin xyz=0 0 0.203 rpy=0 0 0 -> xyz=0 0 0.0 rpy=0 0 0

Commit message: pana

File: src/rrm_cv3_kocur/urdf/arm.urdf (robot description, URDF)
Before this commit: robot arm, 10 links, 9 joints
Joints:
- joint link1_to_joint_1: origin xyz=0 0 0.0 rpy=0 0 0 -> xyz=0 0 0.1015 rpy=0 0 0

Commit message: david urdf

File: src/rrm_cv3_kocur/urdf/arm.urdf (robot description, URDF)
Before this commit: robot arm, 10 links, 9 joints
Links:
- link joint_3: geometry visual cylinder length=0.1 radius=0.02
- link link2: geometry visual cylinder length=0.220 radius=0.01
Joints:
- joint joint_2: axis 0 0 1 -> 0 1 0; origin xyz=0 0 0 rpy=0 0 0 -> xyz=0 0 0.203 rpy=0 0 0
- joint joint_3: limit lower=-0.178 upper=0 effort=1000.0 velocity=0.5 -> lower=-0.1 upper=0.06 effort=1000.0 velocity=0.5; origin xyz=0 0 0 rpy=0 0 0 -> xyz=0 0 0.178 rpy=0 0 0
- joint joint_4: limit lower=-1.62 upper=1.62 effort=1000.0 velocity=0.5 -> lower=-0.96 upper=2.182 effort=1000.0 velocity=0.5; origin xyz=0 0 0 rpy=0 0 0 -> xyz=0 0 0.178 rpy=0 0 0
- joint joint_4_to_tool0: origin xyz=0 0 0 rpy=0 0 0 -> xyz=0 0 0.178 rpy=0 0 0

Commit message: mine back

File: src/rrm_cv3_kocur/urdf/arm.urdf (robot description, URDF)
Before this commit: robot arm, 10 links, 9 joints
Links:
- link joint_3: geometry visual sphere radius=0.03
- link link2: geometry visual cylinder length=0.178 radius=0.01
Joints:
- joint joint_2: axis 0 1 0 -> 0 0 1; origin xyz=0 0 0.203 rpy=0 0 0 -> xyz=0 0 0 rpy=0 0 0
- joint joint_3: limit lower=-0.1 upper=0.06 effort=1000.0 velocity=0.5 -> lower=-0.178 upper=0 effort=1000.0 velocity=0.5; origin xyz=0 0 0.178 rpy=0 0 0 -> xyz=0 0 0 rpy=0 0 0
- joint joint_4: limit lower=-0.96 upper=2.182 effort=1000.0 velocity=0.5 -> lower=-1.62 upper=1.62 effort=1000.0 velocity=0.5; origin xyz=0 0 0.178 rpy=0 0 0 -> xyz=0 0 0 rpy=0 0 0
- joint joint_4_to_tool0: origin xyz=0 0 0.178 rpy=0 0 0 -> xyz=0 0 0 rpy=0 0 0
