Commit message: kar

File: src/abb_config/config/gazebo_abb_irb4600_20_250.urdf (robot description, URDF)
Before this commit: robot abb_irb4600_20_250, 10 links, 9 joints
Links:
- added link kar, mass 0.1; collision mesh filename=package://abb_config/tool.stl; visual mesh filename=package://abb_config/tool.stl
Joints:
- added joint tool0-kar: type fixed, parent tool0, child kar, origin xyz=0 0 0 rpy=0 1.5707963267948966 0

Commit message: link6 kar

File: src/abb_config/config/gazebo_abb_irb4600_20_250.urdf (robot description, URDF)
Before this commit: robot abb_irb4600_20_250, 11 links, 10 joints
Joints:
- removed joint tool0-kar
- added joint link_6-kar: type fixed, parent link_6, child kar, origin xyz=0 0 0 rpy=0 0 0

Commit message: back

File: src/abb_config/config/gazebo_abb_irb4600_20_250.urdf (robot description, URDF)
Before this commit: robot abb_irb4600_20_250, 11 links, 10 joints
Links:
- removed link kar
Joints:
- removed joint link_6-kar

Commit message: cudak

File: src/abb_config/config/gazebo_abb_irb4600_20_250.urdf (robot description, URDF)
Before this commit: robot abb_irb4600_20_250, 10 links, 9 joints
Links:
- added link link_7; visual cylinder length=0.15 radius=0.01
Joints:
- added joint link6_to_link7: type fixed, parent link6, child link7, origin xyz=0 0 0 rpy=0 0 0

Commit message: _ kurwa

File: src/abb_config/config/gazebo_abb_irb4600_20_250.urdf (robot description, URDF)
Before this commit: robot abb_irb4600_20_250, 11 links, 10 joints
Joints:
- removed joint link6_to_link7
- added joint link_6_to_link_7: type fixed, parent link_6, child link_7, origin xyz=0 0 0 rpy=0 0 0

Commit message: back

File: src/abb_config/config/gazebo_abb_irb4600_20_250.urdf (robot description, URDF)
Before this commit: robot abb_irb4600_20_250, 11 links, 10 joints
Links:
- removed link link_7
Joints:
- removed joint link_6_to_link_7
